Commit message: Fix boot submodule sync on fresh clones; set provisional lidar mount
startup.sh: a bare 'git submodule update' aborts on the repo's orphaned
gitlinks (librealsense, ublox_dgnss, sim/src/serial) before fetching
sllidar_ros2, so a fresh Pi clone never got the driver. Update only the
paths registered in .gitmodules.

robot_description: lidar centred on the robot, 1.5 ft above the bottom of
base_link (z = 0.357 from the chassis centre). Provisional until TDM-13.

Co-Authored-By: Claude Opus 5.5 <noreply@anthropic.com>
Claude-Session: https://claude.ai/code/session_01DbW97hUAn6A8RHwzgBycwz

File: ros2_ws/src/robot_description/urdf/robot.urdf.xacro (robot description, xacro)
@@ -15,10 +15,14 @@
   <!-- ===================== Sensor mounts (edit these) ===================== -->
   <!-- Offsets are from base_link (chassis centre), metres / radians.         -->
-  <!-- TODO(TDM-13): replace with measured values.
-       Placeholders are the sim's values: x = chassis_length/2 - 0.1,
-       z = chassis_height/2 + 0.05. -->
-  <xacro:property name="lidar_x" value="0.3"/>
+  <!-- Provisional mount (2026-09-25, not final): centred on the robot, and
+       1.5 ft (0.4572 m) above the BOTTOM of base_link. base_link is the chassis
+       centre and the chassis is chassis_height (0.2 m) tall, so its bottom is
+       at z = -0.10 and the lidar is at z = 0.4572 - 0.10 = 0.357.
+       lidar_link should be the scan plane (optical centre, roughly mid-height
+       of the C1's spinning head): if the 1.5 ft is to the C1's base instead,
+       add ~0.02. Final numbers + yaw come from TDM-13 / TDM-15. -->
+  <xacro:property name="lidar_x" value="0.0"/>
   <xacro:property name="lidar_y" value="0.0"/>
-  <xacro:property name="lidar_z" value="0.15"/>
+  <xacro:property name="lidar_z" value="0.357"/>
   <xacro:property name="lidar_yaw" value="0.0"/>
   <!-- TODO(TDM-13): replace with measured values.

Commit message: TDM-3: camera mount as camera_x/y/z/pitch/yaw xacro properties
camera_link is now the RealSense driver's root frame, placed by editable
mount properties. The driver hangs camera_*_optical_frame off it.
Provisional values keep the old placeholder pose until TDM-6 measures it.

Co-Authored-By: Claude Opus 5.5 <noreply@anthropic.com>

File: ros2_ws/src/robot_description/urdf/robot.urdf.xacro (robot description, xacro)
@@ -7,5 +7,7 @@
                                 -> imu_link     (imu_node stamps this, fixed)
                                 -> gps_link     (fixed)
-                                -> camera_link  (fixed, optional)
+                                -> camera_link  (RealSense mount, fixed; the
+                                                 driver adds camera_link ->
+                                                 camera_*_optical_frame)
                                 -> *_wheel / *_steering_link (moving joints)
   Moving joints (wheels, steering) only get TF once something publishes
@@ -32,4 +34,18 @@
   <xacro:property name="imu_z" value="0.1"/>
   <xacro:property name="imu_yaw" value="0.0"/>
+  <!-- Intel RealSense depth camera. camera_link is the RealSense driver's own
+       root frame (x forward, y left, z up; origin at the depth module's left
+       imager, ~1.75 cm left of the camera body's centre on a D435). The driver
+       publishes camera_link -> camera_{depth,color}_optical_frame, so the pose
+       here is the only mount calibration. pitch > 0 tilts the camera DOWN
+       (REP-103: +pitch about +y).
+       Provisional (2026-09-26): same pose the placeholder camera_link had
+       (front edge of the chassis, 0.15 m above base_link, level). Measured
+       values come from TDM-6. -->
+  <xacro:property name="camera_x" value="0.4"/>
+  <xacro:property name="camera_y" value="0.0"/>
+  <xacro:property name="camera_z" value="0.15"/>
+  <xacro:property name="camera_pitch" value="0.0"/>
+  <xacro:property name="camera_yaw" value="0.0"/>
   <!-- ============================ Chassis ================================= -->
   <xacro:property name="chassis_length" value="0.8"/>
@@ -172,5 +188,5 @@
     <parent link="base_link"/>
     <child link="camera_link"/>
-    <origin xyz="${chassis_length/2} 0 0.15" rpy="0 0 0"/>
+    <origin xyz="${camera_x} ${camera_y} ${camera_z}" rpy="0 ${camera_pitch} ${camera_yaw}"/>
   </joint>
 </robot>

Commit message: TDM-3: provisional camera mount in front of and above the chassis
Eyeballed with the user: ~5 cm past the chassis front edge (x 0.40 -> 0.45)
and ~5 cm above its top (z 0.15), level. Laptop test with the D435i gives
base_link -> camera_depth_optical_frame = (0.45, 0, 0.15) and a single TF
tree. Measured values still come from TDM-6.

Co-Authored-By: Claude Opus 5.5 <noreply@anthropic.com>
Claude-Session: https://claude.ai/code/session_01MFkc7uFzQQf812jwr1m3ob

File: ros2_ws/src/robot_description/urdf/robot.urdf.xacro (robot description, xacro)
@@ -40,8 +40,8 @@
        here is the only mount calibration. pitch > 0 tilts the camera DOWN
        (REP-103: +pitch about +y).
-       Provisional (2026-09-26): same pose the placeholder camera_link had
-       (front edge of the chassis, 0.15 m above base_link, level). Measured
-       values come from TDM-6. -->
-  <xacro:property name="camera_x" value="0.4"/>
+       Provisional (2026-09-26, eyeballed): slightly in front of and above the
+       chassis box, i.e. ~5 cm past its front edge (x = 0.40) and ~5 cm above
+       its top (z = 0.10), level. Measured values come from TDM-6. -->
+  <xacro:property name="camera_x" value="0.45"/>
   <xacro:property name="camera_y" value="0.0"/>
   <xacro:property name="camera_z" value="0.15"/>

Commit message: TDM-20: root the URDF at base_link, base_footprint as its child
The EKF publishes odom -> base_link, so the URDF's base_footprint ->
base_link gave base_link two TF parents; tf2 kept odom and orphaned
base_footprint, and every lookup through it (depth_obstacles'
ground_frame) failed once the EKF ran.

base_joint is now base_link -> base_footprint at z = -wheel_radius
(-0.15); every other offset is unchanged. base_footprint still sits on
the ground, so ground_frame: base_footprint keeps working.

Checked on ROS_DOMAIN_ID=72 with robot_state_publisher + a fake 10 Hz
odom -> base_link broadcaster: base_footprint -> lidar_link = (0, 0,
0.507) and odom -> base_footprint = (x, y, -0.15) both resolve (main's
URDF: ConnectivityException for both).

Updated the comments that described the chain as base_footprint ->
base_link (description launch, package.xml, costmap_lidar.example.yaml,
realsense.yaml, master_launch.py, deployment/README.md) and noted the
expected, harmless KDL "root link has an inertia" warning.

Co-Authored-By: Claude Opus 5.5 <noreply@anthropic.com>
Claude-Session: https://claude.ai/code/session_019uGWZBNY4vkvV4wHR6a1at

File: ros2_ws/src/robot_description/urdf/robot.urdf.xacro (robot description, xacro)
@@ -4,11 +4,16 @@
   Ported from delivery-autonomy/src/simulation/urdf/robot.urdf.xacro with all
   <gazebo> tags/plugins removed, so sim and real share the same frame names:
-    base_footprint -> base_link -> lidar_link   (scan frame, fixed)
-                                -> imu_link     (imu_node stamps this, fixed)
-                                -> gps_link     (fixed)
-                                -> camera_link  (RealSense mount, fixed; the
-                                                 driver adds camera_link ->
-                                                 camera_*_optical_frame)
-                                -> *_wheel / *_steering_link (moving joints)
+    base_link -> base_footprint (ground under the chassis centre, fixed)
+              -> lidar_link     (scan frame, fixed)
+              -> imu_link       (imu_node stamps this, fixed)
+              -> gps_link       (fixed)
+              -> camera_link    (RealSense mount, fixed; the driver adds
+                                 camera_link -> camera_*_optical_frame)
+              -> *_wheel / *_steering_link (moving joints)
+  base_link is the ROOT link because the delivery-autonomy EKF publishes
+  odom -> base_link. A URDF base_footprint -> base_link would give base_link
+  two TF parents and orphan base_footprint (every lookup through it fails).
+  base_footprint hangs wheel_radius below base_link, so z = 0 in it is the
+  ground (depth_obstacles' ground_frame).
   Moving joints (wheels, steering) only get TF once something publishes
   /joint_states; the fixed sensor frames above are unaffected.
@@ -74,5 +79,4 @@
     </inertial>
   </xacro:macro>
-  <link name="base_footprint"/>
   <link name="base_link">
     <visual>
@@ -89,8 +93,15 @@
     <xacro:box_inertia m="${chassis_mass}" w="${chassis_width}" h="${chassis_height}" d="${chassis_length}"/>
   </link>
+  <!-- base_footprint is a CHILD of base_link (see the header): the EKF owns
+       odom -> base_link, so base_link must be the URDF root.
+       Expected startup WARN from robot_state_publisher: "root link base_link
+       has an inertia ... KDL does not support". Harmless (KDL ignores the
+       root inertia; nothing simulates this model). Do NOT add a dummy root
+       link above base_link to silence it: that is the double-parent bug. -->
+  <link name="base_footprint"/>
   <joint name="base_joint" type="fixed">
-    <parent link="base_footprint"/>
-    <child link="base_link"/>
-    <origin xyz="0 0 ${wheel_radius}" rpy="0 0 0"/>
+    <parent link="base_link"/>
+    <child link="base_footprint"/>
+    <origin xyz="0 0 ${-wheel_radius}" rpy="0 0 0"/>
   </joint>
   <!-- ============================= Wheels ================================= -->
