File: PCB/Robotics.kicad_pcb (KiCad board)
At the start: 2 copper layers, 100 x 100 mm, 26 parts, among them J1 XT60PW-F, J13 1x22 female 2.54mm, J14 1x22 female 2.54mm, J15 Micro-Fit 2x4, J16 D36V50F5, J17 JST-SH 4P, J2 XT60PW-F, J3 XT60PW-F, J4 XT60PW-F, J5 JST-GH 4P, J9 XT90PW-M, U2 SN65HVD230

Commit message: Completed PCB Layout
Parts:
- moved F4 16.2 mm to (135.0, 68.5), turned to 90 degrees
- moved F3 14.7 mm to (135.0, 91.0), turned to 90 degrees
- moved J17 7.83 mm to (203.5, 105.5)
- moved J5 6.20 mm to (203.3, 91.4)
- moved NT1 3.91 mm to (196.0, 111.0), turned to 90 degrees
- moved F2 3.00 mm to (137.5, 104.0)
- moved J2 2.12 mm to (126.7, 100.4)
- moved J3 2.06 mm to (126.7, 80.9)
- moved J4 2.06 mm to (126.7, 60.4)
- moved F1 2.00 mm to (137.5, 127.5)
- moved J1 1.95 mm to (126.7, 121.2)
- moved C3 1.84 mm to (182.5, 103.0), turned to 90 degrees
Connections:
- J13 pad 10: /5V Logic and Sensors/ESP_RX_PI_TX -> /5V Logic and Sensors/ESP_TX_PI_RX
- J13 pad 11: /5V Logic and Sensors/ESP_TX_PI_RX -> /5V Logic and Sensors/ESP_RX_PI_TX
- J15 pad 6: /5V Logic and Sensors/ESP_TX_PI_RX -> /5V Logic and Sensors/ESP_RX_PI_TX
- J15 pad 8: /5V Logic and Sensors/ESP_RX_PI_TX -> /5V Logic and Sensors/ESP_TX_PI_RX
Routing:
- net +5V: track 0.00 -> 92.0 mm
- net /5V Logic and Sensors/VBAT_LOGIC: track 0.00 -> 74.8 mm
- net +3.3V: track 0.00 -> 39.5 mm, vias 0 -> 2
- net /5V Logic and Sensors/PI_SDA: track 0.00 -> 32.8 mm, vias 0 -> 3
- net /5V Logic and Sensors/ESP_TX_PI_RX: track 0.00 -> 31.9 mm, vias 0 -> 2
- net /5V Logic and Sensors/PI_SCL: track 0.00 -> 25.3 mm, vias 0 -> 2
- net /Motor Distribution/CAN_L: track 0.00 -> 23.2 mm
- net /5V Logic and Sensors/CAN_RX: track 0.00 -> 22.6 mm, vias 0 -> 4
- net /Motor Distribution/CAN_H: track 0.00 -> 20.8 mm, vias 0 -> 2
- net /5V Logic and Sensors/ESP_RX_PI_TX: track 0.00 -> 20.5 mm, vias 0 -> 2
- net /5V Logic and Sensors/CAN_TX: track 0.00 -> 17.8 mm, vias 0 -> 2
- net /Motor Distribution/GND_PWR: track 0.00 -> 11.8 mm, vias 0 -> 3
- net GND: vias 0 -> 10
- added copper zone on F.Cu, net /5V Logic and Sensors/VBAT_LOGIC
- added copper zone on B.Cu, net /Motor Distribution/GND_PWR
- added copper zone on F.Cu, net /Motor Distribution/VBAT_MOTOR
- added copper zone on F.Cu, net /Motor Distribution/VM1
- added copper zone on F.Cu, net /Motor Distribution/VM2
- added copper zone on F.Cu, net /Motor Distribution/VM3
- added copper zone on F.Cu, net /Motor Distribution/VM4
- added copper zone on B.Cu, net GND
- added copper zone on F.Cu, net GND
Other:
- board text added: "+ BATT -"
- board text added: "120Ω DIP"
- board text added: "20A FUSE"
- board text added: "5A FUSE"
- board text added: "CAN TO ODRIVE 1"
- board text added: "Delivery Bot Power Board Rev A 2026-10"
- board text added: "IMU"
- board text added: "ODRIVE 1"
- board text added: "ODRIVE 2"
- board text added: "ODRIVE 3"
- board text added: "ODRIVE 4"
- board text added: "RPI"
- board text added: "VIN"
- board text added: "VOUT"
