File: PCB/sensor.kicad_sch (KiCad schematic)
At the start: 10 parts, among them J13 1x22 female 2.54mm, J14 1x22 female 2.54mm, J15 Micro-Fit 2x4, J16 D36V50F5, J17 JST-SH 4P, U2 SN65HVD230

Commit message: Completed PCB Layout
Connections:
- net ESP_RX_PI_TX: now also J13.11 (Pin_11), J15.6 (Pin_6); no longer J13.10 (Pin_10), J15.8 (Pin_8)
- net ESP_TX_PI_RX: now also J13.10 (Pin_10), J15.8 (Pin_8); no longer J13.11 (Pin_11), J15.6 (Pin_6)
Changed lines of the file:
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@@
 		)
 	)
-	(label "ESP_TX_PI_RX"
+	(label "ESP_RX_PI_TX"
 		(at 245.11 95.25 0)
 		(effects
@@
 		)
 	)
-	(label "ESP_RX_PI_TX"
+	(label "ESP_TX_PI_RX"
 		(at 133.35 49.53 180)
 		(effects
@@
 		)
 	)
-	(label "ESP_RX_PI_TX"
+	(label "ESP_TX_PI_RX"
 		(at 245.11 97.79 0)
 		(effects
@@
 		)
 	)
-	(label "ESP_TX_PI_RX"
+	(label "ESP_RX_PI_TX"
 		(at 133.35 52.07 180)
 		(effects
